File: MiSTdon.kicad/MiSTdon.kicad_pcb (KiCad board)
At the start: 2 copper layers, 70 x 70 mm, 32 parts, among them J1 Conn_02x06_Top_Bottom, J10 Conn_01x03, J11 Conn_01x05, J2 Conn_01x12, J3 Conn_01x05, J4 Conn_02x10_Odd_Even, J5 Conn_02x10_Odd_Even, J6 Conn_02x03_Odd_Even, J7 Conn_02x06_Top_Bottom, J8 DB9_Male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

Commit message: Kicad done, missing routing
Parts:
- J11: value Conn_01x05 -> Conn_01x06; footprint Connector_PinHeader_2.54mm:PinHeader_1x05_P2.54mm_Vertical -> Connector_PinHeader_2.54mm:PinHeader_1x06_P2.54mm_Vertical
- JP3: value Conn_01x02 -> Conn_01x03; footprint Connector_PinHeader_2.54mm:PinHeader_1x02_P2.54mm_Vertical -> Connector_PinHeader_2.54mm:PinHeader_1x03_P2.54mm_Vertical
- moved JP2 19.2 mm to (130.2, 82.5)
- moved R3 14.8 mm to (143.5, 94.3), turned to 90 degrees
- moved R4 6.10 mm to (154.0, 54.0), turned to 0 degrees
- moved R12 5.40 mm to (141.7, 112.4)
- moved J11 5.09 mm to (166.4, 83.2)
- moved JP5 4.45 mm to (149.9, 82.5)
- moved JP4 3.68 mm to (146.1, 67.9), turned to 90 degrees
- moved R10 2.55 mm to (166.4, 103.7)
- moved R9 2.55 mm to (166.4, 100.1)
- moved R11 2.55 mm to (166.4, 106.7)
- moved SW1 2.53 mm to (134.9, 56.1)
- moved D1 1.77 mm to (141.7, 116.2)
- moved J6 1.27 mm to (120.7, 110.5)
- moved JP3 0.90 mm to (134.6, 67.9)
- moved R1 0.64 mm to (159.4, 108.6), turned to 180 degrees
Other:
- board text added: "D0"
- board text added: "DBG"
- board text added: "DISK"
- board text added: "MI"
- board text added: "MO"
- board text added: "S2"
- board text added: "S3"
- board text added: "S4"
- board text added: "SCK"
- board text added: "SW2"
- board text removed: "SW2 DBG"

Commit message: v0.7 PCB gerbers generated for manufacturing
Parts:
- added LO2: OSHW-Logo2_14.6x12mm_SilkScreen, Symbol:OSHW-Logo2_14.6x12mm_SilkScreen, F.Cu at (123.8, 66.0)
- added LO4: ESD-Logo_6.6x6mm_SilkScreen, Symbol:ESD-Logo_6.6x6mm_SilkScreen, B.Cu at (142.2, 114.9)
- added REF**: KiCad-Logo2_5mm_SilkScreen, Symbol:KiCad-Logo2_5mm_SilkScreen, B.Cu at (124.1, 63.6)
- moved R11 0.76 mm to (166.4, 107.4)
- turned R2 to -90 degrees
Connections:
- net /PB2_AD6 renamed /PB2_AD6_OSD
- net /PB3_AD7 renamed /PB3_AD7_USER
Routing:
- net /3V3: track 0.00 -> 153.3 mm, vias 0 -> 3
- net /NRST2: track 0.00 -> 102.6 mm, vias 0 -> 3
- net /NRST: track 0.00 -> 94.6 mm
- net /PA4_CONF_DONE: track 0.00 -> 75.1 mm, vias 0 -> 3
- net /PA8_CONF_NCFG: track 0.00 -> 72.8 mm, vias 0 -> 1
- net /PA18_J0B1: track 0.00 -> 71.3 mm
- net /PA7_CONF_NSTAT: track 0.00 -> 70.9 mm, vias 0 -> 2
- net /PA9_CONF_D0: track 0.00 -> 64.4 mm
- net /5V: track 0.00 -> 61.6 mm
- net /PA22_J0UP: track 0.00 -> 60.9 mm
- net /PA19_J0RG: track 0.00 -> 60.7 mm, vias 0 -> 1
- net /PA17_J0B2: track 0.00 -> 60.4 mm, vias 0 -> 1
- net /PA23_J1B2: track 0.00 -> 60.2 mm, vias 0 -> 1
- net /PA20_J0LF: track 0.00 -> 59.3 mm
- net /PA21_J0DW: track 0.00 -> 58.3 mm, vias 0 -> 1
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- added copper zone on B.Cu, net GND
- added copper zone on F.Cu, net GND
Other:
- rule pad_to_mask_clearance: 0 -> 0.05
- board text added: "0.1270 mm / 0.1270 mm"
- board text added: "0.3000 mm"
- board text added: "1.6000 mm"
- board text added: "2"
- board text added: "70.0000 mm x 70.0000 mm"
- board text added: "BEFORE USE READ THE README AT https://github.com/somhi/MiSTdon"
- board text added: "BOARD CHARACTERISTICS"
- board text added: "Board Thickness:"
- board text added: "Board overall dimensions:"
- board text added: "Castellated pads:"
- board text added: "Copper Finish:"
- board text added: "Copper Layer Count:"
- board text added: "Edge card connectors:"
- board text added: "Impedance Control:"
- board text added: "MiSTdon v${VERSION}"
- board text added: "Min hole diameter:"
- board text added: "Min track/spacing:"
- board text added: "No"
- board text added: "None"
- board text added: "Plated Board Edge:"

Commit message: v0.8 some changes after testing first PCB
Parts:
- R4: value 4k7 -> 10k
- moved LO4 37.4 mm to (105.2, 109.9)
- moved REF** 3.91 mm to (126.4, 60.5)
- moved J6 2.29 mm to (118.4, 110.5)
Routing:
- net /NRST: track 94.6 -> 92.0 mm
- net /3V3: track 153.3 -> 155.6 mm
Other:
- board text added: "GD"
- board text added: "JTAG SIDE"
- board text added: "RTFM:) BEFORE USE READ https://github.com/somhi/MiSTdon"
- board text added: "USB SIDE"
- board text removed: "BEFORE USE READ THE README AT https://github.com/somhi/MiSTdon"
